File: byggern.sch (KiCad schematic (older format))
At the start: 41 parts, among them J1 Power_Rail, J2 JTAG LINK, J3 OLED_Connection, J4 CAN, J5 P1000 Header, J6 DB9_Female_MountingHoles, U1 Barrel_jack, U10 MAX233, U2 LM340SX, U3 ATmega162-16PU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

Commit message: Change footprints of ICs to DIPs and Close to finish routing
Parts:
- U10: footprint byggern:MAX233CPP -> Package_DIP:DIP-20_W7.62mm_Socket
- U3: footprint Package_DIP:DIP-40_W15.24mm -> Package_DIP:DIP-40_W15.24mm_Socket
- U4: footprint byggern:GAL16V8 -> Package_DIP:DIP-20_W7.62mm_Socket
- U5: footprint byggern:MCP2515-EP -> Package_DIP:DIP-18_W7.62mm_Socket
- U6: footprint byggern:SN74ALS573CN -> Package_DIP:DIP-20_W7.62mm_Socket
- U7: footprint byggern:MCP2551-IP -> Package_DIP:DIP-8_W7.62mm_Socket
- U8: footprint byggern:CY7C185-20PC -> Package_DIP:DIP-28_W7.62mm_Socket
- U9: footprint byggern:ADC0844CCN -> Package_DIP:DIP-20_W7.62mm_Socket
- Y1, Y2: footprint Connector_PinHeader_2.54mm:PinHeader_1x02_P2.54mm_Vertical -> Crystal:Crystal_SMD_HC49-SD_HandSoldering
Changed lines of the file:
@@
 F 0 "Y1" V 954 2381 50  0000 L CNN
 F 1 "4.9MHz" V 1045 2381 50  0000 L CNN
-F 2 "Connector_PinHeader_2.54mm:PinHeader_1x02_P2.54mm_Vertical" H 1000 2250 50  0001 C CNN
+F 2 "Crystal:Crystal_SMD_HC49-SD_HandSoldering" H 1000 2250 50  0001 C CNN
 F 3 "~" H 1000 2250 50  0001 C CNN
 	1    1000 2250
@@
 F 0 "U3" H 2200 5700 50  0000 C CNN
 F 1 "ATmega162-16PU" H 2500 5600 50  0000 C CNN
-F 2 "Package_DIP:DIP-40_W15.24mm" H 2100 3650 50  0001 C CIN
+F 2 "Package_DIP:DIP-40_W15.24mm_Socket" H 2100 3650 50  0001 C CIN
 F 3 "http://ww1.microchip.com/downloads/en/DeviceDoc/Atmel-2513-8-bit-AVR-Microntroller-ATmega162_Datasheet.pdf" H 2100 3650 50  0001 C CNN
 	1    2100 3650
@@
 F 0 "U10" H 10000 3450 50  0000 C CNN
 F 1 "MAX233" H 10100 3350 50  0000 C CNN
-F 2 "byggern:MAX233CPP" H 9300 3450 50  0001 C CNN
+F 2 "Package_DIP:DIP-20_W7.62mm_Socket" H 9300 3450 50  0001 C CNN
 F 3 "" H 9300 3450 50  0001 C CNN
 	1    9550 3650
@@
 F 0 "U4" H 4450 4950 50  0000 C CNN
 F 1 "GAL16V8" H 4550 4850 50  0000 C CNN
-F 2 "byggern:GAL16V8" H 4350 4250 50  0001 C CNN
+F 2 "Package_DIP:DIP-20_W7.62mm_Socket" H 4350 4250 50  0001 C CNN
 F 3 "" H 4350 4250 50  0001 C CNN
 	1    4350 4250
@@
 F 0 "U8" H 7050 2850 50  0000 L CNN
 F 1 "IDT7164" H 7050 2750 50  0000 L CNN
-F 2 "byggern:CY7C185-20PC" H 6700 3150 50  0001 C CNN
+F 2 "Package_DIP:DIP-28_W7.62mm_Socket" H 6700 3150 50  0001 C CNN
 F 3 "" H 6700 3150 50  0001 C CNN
 	1    6700 2050
@@
 F 0 "U6" H 5700 1650 50  0000 C CNN
 F 1 "SN74ALS573CN" H 5900 1550 50  0000 C CNN
-F 2 "byggern:SN74ALS573CN" H 5450 1450 50  0001 C CNN
+F 2 "Package_DIP:DIP-20_W7.62mm_Socket" H 5450 1450 50  0001 C CNN
 F 3 "" H 5450 1450 50  0001 C CNN
 	1    5450 1400
@@
 F 0 "U9" H 8750 1450 50  0000 C CNN
 F 1 "ADC0844" H 8850 1350 50  0000 C CNN
-F 2 "byggern:ADC0844CCN" H 8800 1350 50  0001 C CNN
+F 2 "Package_DIP:DIP-20_W7.62mm_Socket" H 8800 1350 50  0001 C CNN
 F 3 "" H 8800 1350 50  0001 C CNN
 	1    8450 1350
@@
 F 0 "U5" H 4900 5650 50  0000 C CNN
 F 1 "MCP2515" H 5050 5550 50  0000 C CNN
-F 2 "byggern:MCP2515-EP" H 4700 5750 50  0001 C CNN
+F 2 "Package_DIP:DIP-18_W7.62mm_Socket" H 4700 5750 50  0001 C CNN
 F 3 "" H 4700 5750 50  0001 C CNN
 	1    4700 5750
@@
 F 0 "Y2" V 3950 7250 50  0000 R CNN
 F 1 "16MHz" V 3850 7250 50  0000 R CNN
-F 2 "Connector_PinHeader_2.54mm:PinHeader_1x02_P2.54mm_Vertical" H 3850 6900 50  0001 C CNN
+F 2 "Crystal:Crystal_SMD_HC49-SD_HandSoldering" H 3850 6900 50  0001 C CNN
 F 3 "~" H 3850 6900 50  0001 C CNN
 	1    3850 6900
@@
 F 0 "U7" H 6600 5150 50  0000 C CNN
 F 1 "MCP2551" H 6700 5050 50  0000 C CNN
-F 2 "byggern:MCP2551-IP" H 6350 5500 50  0001 C CNN
+F 2 "Package_DIP:DIP-8_W7.62mm_Socket" H 6350 5500 50  0001 C CNN
 F 3 "" H 6350 5500 50  0001 C CNN
 	1    6350 5500

Commit message: Fix errors and update BOM
Parts:
- removed J2: JTAG LINK, Connector_PinHeader_2.54mm:PinHeader_1x04_P2.54mm_Vertical, symbol Connector_Generic:Conn_01x04
- removed J6: DB9_Female_MountingHoles, Connector_Dsub:DSUB-9_Female_Vertical_P2.77x2.84mm_MountingHoles, symbol Connector:DB9_Female_MountingHoles
- removed R6: 120, Resistor_SMD:R_0805_2012Metric_Pad1.15x1.40mm_HandSolder, symbol Device:R_Small
- added J2: JTAG LINK, Connector_PinHeader_2.54mm:PinHeader_2x04_P2.54mm_Vertical, symbol Connector_Generic:Conn_02x04_Odd_Even
- added J6: A-DF_09_A_KG-T2S, digikey-footprints:DSUB-9_Receptical_A-DF_09_A_KG-T2S, symbol dk_D-Sub-Connectors:A-DF_09_A_KG-T2S
- added TP1, TP10, TP11, TP12, TP2, TP3, TP4, TP5, TP6, TP7, TP8, TP9: TestPoint, TestPoint:TestPoint_Pad_D1.5mm, symbol Connector:TestPoint
Connections:
- net A10: now also U4.2 (I2); no longer U4.3 (I3)
- net A11: now also U4.1 (I1/CLK); no longer U4.4 (I4)
- net A8: now also U4.4 (I4); no longer U4.1 (I1/CLK)
- net A9: now also U4.3 (I3); no longer U4.2 (I2)
- net CAN_~INT~: now also TP7.1
- net GND: now also U8.20 (~CS~1), J2.6 (Pin_6), J2.8 (Pin_8), J6.10, J6.5
- net LE: now also TP10.1
- net RXD_232: now also TP5.1
- net SCK: now also TP4.1
- net TXD_232: now also TP6.1
- net VCC: now also J2.2 (Pin_2); no longer U8.26 (CS2)
- net ~CS~_ADC: now also TP12.1
- net ~CS~_MCP: now also TP3.1
- net ~OE~: now also TP9.1
- net ~RESET~: now also TP2.1
- net ~WR~: now also TP8.1
- net at U3.25 (PC4): now also J2.1 (Pin_1)
- net at U3.26 (PC5): now also J2.3 (Pin_3)
- net at U3.27 (PC6): now also J2.5 (Pin_5)
- net at U3.28 (PC7): now also J2.7 (Pin_7)
- net ADC_~INT~: now reaches U3.31 (PE0)
- net ADC_~INT~: now also U9.18 (~INTR), TP1.1
- net TO3: now reaches U10.4 (R1IN)
- net TO3: now also J6.3
- net TO2: now reaches U10.5 (T1OUT)
- net TO2: now also J6.2
- net ~CS~_RAM renamed CS_RAM
- net CS_RAM: now also U8.26 (CS2), TP11.1; no longer U8.20 (~CS~1)
- no-connect marks 38 -> 37
Other:
- moved on the sheet: C15, R5, U10
